File: vtx-scanner-pcb/vtx-scanner-pcb.sch (KiCad schematic (older format))
At the start: 31 parts, among them CON1 SJ-3523-SMT-TR, J1 Conn_01x06_Male, J2 Conn_01x08_Female, J3 SMA-J-P-H-RA-TH1, J4 Conn_01x05, J5 XT60-M, Q1 MMSS8050-H-TP, Q2 MMSS8050-H-TP, Q3 MMSS8050-H-TP, U1 RX5808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

Commit message: Minor update in schematic
Other:
- note added: "Replaced with NCV1117"
Changed lines of the file:
@@
 Text Notes 4950 3800 2    50   ~ 0
 strapping pin\n
+Text Notes 1450 2750 0    50   ~ 0
+Replaced with NCV1117
 $EndSCHEMATC

Commit message: Reworked PCB
 - missing pullups IO0/EN
 - added capacitors for EN
 - clearance around mounting holes
 - better 2.4GHz antenna placement
 - correct rx5808 size
Parts:
- removed J2: Conn_01x08_Female, Connector_PinHeader_2.54mm:PinHeader_1x08_P2.54mm_Horizontal, symbol Connector:Conn_01x08_Female
- added J2: sh1106-1.3inch-oled, deets:sh1106-1.3inch-oled, symbol deets:sh1106-1.3inch-oled
- CON1: symbol dk_Barrel-Audio-Connectors:SJ-3523-SMT-TR -> vtx-scanner-pcb-rescue:SJ-3523-SMT-TR-dk_Barrel-Audio-Connectors
- Q1, Q2, Q3: symbol dk_Transistors-Bipolar-BJT-Single:MMSS8050-H-TP -> vtx-scanner-pcb-rescue:MMSS8050-H-TP-dk_Transistors-Bipolar-BJT-Single
- S1, S2, S3, S4: symbol dk_Tactile-Switches:FSM4JSMATR -> vtx-scanner-pcb-rescue:FSM4JSMATR-dk_Tactile-Switches
Connections:
- net +3V3: now also J2.2 (VCC)
- net -BATT: now also J2.1 (GND)
- net SSD1306_CLK: now also J2.3 (CLK)
- net SSD1306_CS: now also J2.7 (CS)
- net SSD1306_DATA: now also J2.4 (MOSI)
- net SSD1306_DC: now also J2.6 (DC)
- net SSD1306_RST: now also J2.5 (RESET)
- no-connect marks 15 -> 14
Changed lines of the file:
@@
 EESchema Schematic File Version 4
 LIBS:vtx-scanner-pcb-cache
-EELAYER 26 0
+EELAYER 29 0
 EELAYER END
 $Descr A4 11693 8268
@@
 NoConn ~ 5000 2800
 $Comp
-L Connector:Conn_01x08_Female J2
-U 1 1 5C69E4E5
-P 7900 4000
-F 0 "J2" H 7927 3976 50  0000 L CNN
-F 1 "Conn_01x08_Female" H 7927 3885 50  0000 L CNN
-F 2 "Connector_PinHeader_2.54mm:PinHeader_1x08_P2.54mm_Horizontal" H 7900 4000 50  0001 C CNN
-F 3 "~" H 7900 4000 50  0001 C CNN
-	1    7900 4000
-	1    0    0    -1
-$EndComp
-Wire Wire Line
-	7700 3700 7350 3700
-$Comp
 L power:GND #PWR014
 U 1 1 5C69EBDF
-P 7350 3700
-F 0 "#PWR014" H 7350 3450 50  0001 C CNN
-F 1 "GND" H 7355 3527 50  0000 C CNN
-F 2 "" H 7350 3700 50  0001 C CNN
-F 3 "" H 7350 3700 50  0001 C CNN
-	1    7350 3700
-	1    0    0    -1
-$EndComp
-NoConn ~ 7700 3800
-Wire Wire Line
-	7700 3900 7550 3900
-Wire Wire Line
-	7550 3900 7550 3600
-Wire Wire Line
-	7550 3600 7350 3600
+P 8250 3000
+F 0 "#PWR014" H 8250 2750 50  0001 C CNN
+F 1 "GND" H 8255 2827 50  0000 C CNN
+F 2 "" H 8250 3000 50  0001 C CNN
+F 3 "" H 8250 3000 50  0001 C CNN
+	1    8250 3000
+	1    0    0    -1
+$EndComp
 $Comp
 L power:+3.3V #PWR013
 U 1 1 5C6A5EDE
-P 7350 3600
-F 0 "#PWR013" H 7350 3450 50  0001 C CNN
-F 1 "+3.3V" H 7365 3773 50  0000 C CNN
-F 2 "" H 7350 3600 50  0001 C CNN
-F 3 "" H 7350 3600 50  0001 C CNN
-	1    7350 3600
-	1    0    0    -1
-$EndComp
-Text Label 7700 4000 2    50   ~ 0
+P 7850 3300
+F 0 "#PWR013" H 7850 3150 50  0001 C CNN
+F 1 "+3.3V" H 7865 3473 50  0000 C CNN
+F 2 "" H 7850 3300 50  0001 C CNN
+F 3 "" H 7850 3300 50  0001 C CNN
+	1    7850 3300
+	1    0    0    -1
+$EndComp
+Text Label 8350 3800 2    50   ~ 0
 SSD1306_CS
-Text Label 7700 4100 2    50   ~ 0
+Text Label 8350 3600 2    50   ~ 0
 SSD1306_RST
-Text Label 7700 4200 2    50   ~ 0
+Text Label 8350 3700 2    50   ~ 0
 SSD1306_DC
-Text Label 7700 4300 2    50   ~ 0
+Text Label 8350 3400 2    50   ~ 0
 SSD1306_CLK
-Text Label 7700 4400 2    50   ~ 0
+Text Label 8350 3500 2    50   ~ 0
 SSD1306_DATA
 NoConn ~ 6200 3100
@@
 BUZZER
 $Comp
-L dk_Transistors-Bipolar-BJT-Single:MMSS8050-H-TP Q2
+L vtx-scanner-pcb-rescue:MMSS8050-H-TP-dk_Transistors-Bipolar-BJT-Single Q2
 U 1 1 5C8D54F9
 P 2400 7000
@@
 $EndComp
 $Comp
-L dk_Transistors-Bipolar-BJT-Single:MMSS8050-H-TP Q1
+L vtx-scanner-pcb-rescue:MMSS8050-H-TP-dk_Transistors-Bipolar-BJT-Single Q1
 U 1 1 5C8D5889
 P 2400 6350
@@
 $EndComp
 $Comp
-L dk_Transistors-Bipolar-BJT-Single:MMSS8050-H-TP Q3
+L vtx-scanner-pcb-rescue:MMSS8050-H-TP-dk_Transistors-Bipolar-BJT-Single Q3
 U 1 1 5C8D798E
 P 5200 6700
@@
 $EndComp
 $Comp
-L dk_Tactile-Switches:FSM4JSMATR S1
+L vtx-scanner-pcb-rescue:FSM4JSMATR-dk_Tactile-Switches S1
 U 1 1 5C8D94E0
 P 10200 5950
@@
 $EndComp
 $Comp
-L dk_Tactile-Switches:FSM4JSMATR S2
+L vtx-scanner-pcb-rescue:FSM4JSMATR-dk_Tactile-Switches S2
 U 1 1 5C8D9681
 P 10200 2950
@@
 $EndComp
 $Comp
-L dk_Tactile-Switches:FSM4JSMATR S3
+L vtx-scanner-pcb-rescue:FSM4JSMATR-dk_Tactile-Switches S3
 U 1 1 5C8D978E
 P 10200 4000
@@
 $EndComp
 $Comp
-L dk_Tactile-Switches:FSM4JSMATR S4
+L vtx-scanner-pcb-rescue:FSM4JSMATR-dk_Tactile-Switches S4
 U 1 1 5C8D9896
 P 10200 4900
@@
 $EndComp
 $Comp
-L dk_Barrel-Audio-Connectors:SJ-3523-SMT-TR CON1
+L vtx-scanner-pcb-rescue:SJ-3523-SMT-TR-dk_Barrel-Audio-Connectors CON1
 U 1 1 5CBA07DB
 P 3600 3700
@@
 Text Notes 1450 2750 0    50   ~ 0
 Replaced with NCV1117
+$Comp
+L deets:sh1106-1.3inch-oled J2
+U 1 1 5D28AE75
+P 8550 3500
+F 0 "J2" H 8769 3561 50  0000 L CNN
+F 1 "sh1106-1.3inch-oled" H 8769 3470 50  0000 L CNN
+F 2 "deets:sh1106-1.3inch-oled" H 8550 3500 50  0001 C CNN
+F 3 "" H 8550 3500 50  0001 C CNN
+	1    8550 3500
+	1    0    0    -1
+$EndComp
+Wire Wire Line
+	8350 3000 8250 3000
+Wire Wire Line
+	8350 3000 8350 3200
+Wire Wire Line
+	7850 3300 8350 3300
 $EndSCHEMATC
